File: controller-pcb-eagle/picade.sch (EAGLE design)
At the start: 38 parts

Commit message: Final Picade PCB layout
Parts:
- removed C4: 0.1µF, adafruit:C-USC0603K
- added C12: cercap-22pF-0603, adafruit:C-USC0603K
- added R10, R9: res-1k-0603, resistor:R-EU_R0603
- added R8: res-10k-0603, resistor:R-EU_R0603
- 16MHZ: value (none) -> xtal-16mhz-5x3.2
- AMPLIFIER: value MAX98306ETD+ -> ic-max98306-tdfn14
- ATMEGA32U4: value ATMEGA32U4-AU -> ic-atmega32u4-tqfp44
- C1, C2, C3: value 1µF -> cercap-1uF-0603
- C10: value 1µF -> cercap-100nF-0603; device resistor:C-EUC0603K -> adafruit:C-USC0603K
- C11: value 0.1µF -> cercap-22pF-0603
- C5: value 0.1µF -> cercap-10uF-0805; device adafruit:C-USC0603K -> resistor:C-EUC0805K
- C6: value 10uF -> cercap-100nF-0603; device resistor:C-EUC0805K -> adafruit:C-USC0603K
- C7: value 0.1µF -> cercap-100nF-0603
- C8: value 22pF -> cercap-100nf-0603
- C9: value 22pF -> cercap-1uF-0603; device adafruit:C-USC0603K -> resistor:C-EUC0603K
- F1: value PTCSMD -> ptc-0.5A-120
- HEADPHONES: value AUDIO-JACK2SMD -> stereo-jack-switched; device SparkFun-Connectors:AUDIO-JACK2SMD -> pimoroni:AUDIO-JACK2SMD
- LINEIN: value (none) -> stereo-jack-noswitch
- PWR: value (none) -> led-white-0805
- R1: value 1kΩ -> res-470k-0603
- R2, R3: value 22Ω -> res-47k-0603
- R4: value 1kΩ -> res-1k-0603
- R5: value 1kΩ -> res-22-0603
- R6: value 10kΩ -> res-22-0603
- R7: value 10kΩ -> res-10k-0603
- RESET: value SWITCH-MOMENTARY-2-SMD-1101NE -> gullwing-switch
- RX: value (none) -> led-orange-0805
- TX: value (none) -> led-green-0805
- USB: value CON-USB-F-MICRO-B -> USB-REVERSE-MICROB; device dp_devices:CON-USB-F-MICRO-B -> pimoroni:USB-REVERSE-MICROB
- renumbered CONTROLLER to ATMEGA32U4, JTAG to ICSP
Connections:
- removed net N$43: HEADPHONES.TIP, LINEIN.LEFT
- net GND: now also C11.1, C12.1, C5.2, C9.2, R1.2, R8.1, USB.GND; no longer C11.2, C4.2, C5.1, C9.1, R7.1, USBUSB.GND
- net N$1: now also C11.2; no longer C8.2
- net N$10: now also R9.2; no longer R4.2
- net N$11: now also R9.1; no longer R4.1
- net N$12: now also R10.1; no longer R5.1
- net N$13: now also R10.2; no longer R5.2
- net N$15: now also USB.VBUS; no longer USBUSB.VUSB
- net N$2: now also R5.2; no longer R2.2
- net N$3: now also R5.1, USB.D-; no longer R2.1, USBUSB.D-
- net N$37: now also C1.1, HEADPHONES.RING, LINEIN.RIGHT, R2.1; no longer C2.1, HEADPHONES.TSH
- net N$38: now also C2.1, HEADPHONES.TIP, LINEIN.LEFT, R3.1; no longer C1.1, HEADPHONES.RSH
- net N$4: now also R6.1, USB.D+; no longer R3.1, USBUSB.D+
- net N$41: now also R8.2; no longer R7.2
- net N$42: now also AMPLIFIER.SHDN, HEADPHONES.RSH, R1.1; no longer HEADPHONES.RING, LINEIN.RIGHT
- net N$5: now also R6.2; no longer R3.2
- net N$6: now also C9.1; no longer C10.1
- net N$7: now also C8.2; no longer C5.2
- net N$8: now also C12.2; no longer C9.2
- net N$9: now also R4.1; no longer R1.1
- net RESET: now also R7.1; no longer R6.1
- net VCC: now also C10.1, C5.1, R2.2, R3.2, R4.2, R7.2; no longer AMPLIFIER.SHDN, C11.1, C4.1, R1.2, R6.2
Other:
- moved on the sheet: AMPLIFIER, C10, C11, C5, C6, C7, C8, C9, LINEIN, R1, R2, R3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
